File: PCB/Kicad/imponatorPower/imponatorPower.kicad_sch (KiCad schematic)
At the start: 29 parts, among them J1 UJ20-C-H-G-SMT-1-P16-TR, J2 Conn_01x02, U1 BQ25172DSGR, U2 MP28164GD-Z

Commit message: Finished the second iteration of the imponatorPower project
Parts:
- removed BT1: 2460, Imported:BAT_2460, symbol Imported:2460
- removed C3, C7: 1uF, Capacitor_SMD:C_0805_2012Metric_Pad1.18x1.45mm_HandSolder, symbol Device:C
- removed C4, C5, C6: 22uF, Capacitor_SMD:C_0805_2012Metric_Pad1.18x1.45mm_HandSolder, symbol Device:C
- removed D1: LED, LED_SMD:LED_0201_0603Metric_Pad0.64x0.40mm_HandSolder, symbol Device:LED
- removed F1: MF-R075, Imported:FUS_MF-R075_BRN, symbol Imported:MF-R075
- removed J1: UJ20-C-H-G-SMT-1-P16-TR, Imported:SAMESKY_UJ20-C-H-G-SMT-1-P16-TR, symbol Imported:UJ20-C-H-G-SMT-1-P16-TR
- removed L1: 1uH, Resistor_THT:R_Bare_Metal_Element_L21.3mm_W4.8mm_P20.30mm, symbol Device:L
- removed R1: 1M, Resistor_SMD:R_1206_3216Metric_Pad1.30x1.75mm_HandSolder, symbol Device:R
- removed R10, R4, R5: 10K, Resistor_SMD:R_1206_3216Metric_Pad1.30x1.75mm_HandSolder, symbol Device:R
- removed R11: 560K, Resistor_SMD:R_1206_3216Metric_Pad1.30x1.75mm_HandSolder, symbol Device:R
- removed R12: 100K, Resistor_SMD:R_1206_3216Metric_Pad1.30x1.75mm_HandSolder, symbol Device:R
- removed R2, R3: 56K, Resistor_SMD:R_1206_3216Metric_Pad1.30x1.75mm_HandSolder, symbol Device:R
- removed R6: 62K +- 1%, Resistor_SMD:R_0603_1608Metric_Pad0.98x0.95mm_HandSolder, symbol Device:R
- removed R7: 1K, Resistor_SMD:R_1206_3216Metric_Pad1.30x1.75mm_HandSolder, symbol Device:R
- removed R8: 24K, Resistor_SMD:R_1206_3216Metric_Pad1.30x1.75mm_HandSolder, symbol Device:R
- removed R9: 103AT-2, Resistor_THT:R_Bare_Metal_Element_L21.3mm_W4.8mm_P20.30mm, symbol Device:R
- removed U1: BQ25172DSGR, Imported:IC_BQ25172DSGR, symbol Imported:BQ25172DSGR
- removed U2: MP28164GD-Z, Imported:QFN-11_MP28164_MNP, symbol Imported:MP28164GD-Z
- C1, C2: value 100nF -> 10uF
Connections:
- net +5VL renamed +5Vout
Other:
- added sheet Buck up (buck.kicad_sch)
- added sheet Charging circuit (charing.kicad_sch)
- added sheet usb-c (usb.kicad_sch)
- note removed: "300mA charging"
- note removed: "Max charging time 8 hours"
- moved on the sheet: C1, C2, H1, H2, J2
